Commit message: added CAD sourced measurements for the description URDF

File: fractal_pad_description/urdf/fractal_pad/fractal_pad_macro.xacro (robot description, xacro)
@@ -5,20 +5,73 @@
   <xacro:macro name="fractal_pad" params="prefix parent *origin">
     <!-- Approximate geometry only; replace with measured CAD when available. -->
-    <link name="${prefix}base_link">
+    <link name="${prefix}fractal_coupler">
+      <xacro:default_inertial />
+      <visual>
+        <geometry>
+          <mesh filename="package://fractal_pad_description/meshes/fractal_pad/visual/fractal_coupler.stl" />
+        </geometry>
+        <material name="grey" />
+      </visual>
+      <collision>
+        <geometry>
+          <mesh filename="package://fractal_pad_description/meshes/fractal_pad/collision/fractal_coupler.stl" />
+        </geometry>
+      </collision>
+    </link>
+    <link name="${prefix}fractal_L1">
       <xacro:default_inertial/>
       <visual>
-        <geometry><cylinder length="0.04" radius="0.05"/></geometry>
-        <material name="black"/>
+        <geometry>
+          <mesh filename="package://fractal_pad_description/meshes/fractal_pad/visual/fractal_L1.stl" />
+        </geometry>
+        <material name="red"/>
       </visual>
-      <collision><geometry><cylinder length="0.04" radius="0.05"/></geometry></collision>
+      <collision>
+        <geometry>
+          <mesh filename="package://fractal_pad_description/meshes/fractal_pad/collision/fractal_L1.stl" />
+        </geometry>
+      </collision>
     </link>
-    <link name="${prefix}motor_link">
+    <link name="${prefix}motor_body">
       <xacro:default_inertial/>
       <visual>
-        <origin xyz="0 0 0.04"/>
-        <geometry><cylinder length="0.08" radius="0.035"/></geometry>
-        <material name="blue"/>
+        <geometry>
+          <mesh filename="package://fractal_pad_description/meshes/fractal_pad/visual/fractal_GM2804.stl" />
+        </geometry>
+        <material name="grey"/>
       </visual>
-      <collision><origin xyz="0 0 0.04"/><geometry><cylinder length="0.08" radius="0.035"/></geometry></collision>
+      <collision>
+        <geometry>
+          <mesh filename="package://fractal_pad_description/meshes/fractal_pad/collision/fractal_GM2804.stl" />
+        </geometry>
+      </collision>
+    </link>
+    <link name="${prefix}fractal_L2">
+      <xacro:default_inertial/>
+      <visual>
+        <geometry>
+          <mesh filename="package://fractal_pad_description/meshes/fractal_pad/visual/fractal_L2.stl" />
+        </geometry>
+        <material name="red"/>
+      </visual>
+      <collision>
+        <geometry>
+          <mesh filename="package://fractal_pad_description/meshes/fractal_pad/collision/fractal_L2.stl" />
+        </geometry>
+      </collision>
+    </link>
+    <link name="${prefix}fractal_L4">
+      <xacro:default_inertial/>
+      <visual>
+        <geometry>
+          <mesh filename="package://fractal_pad_description/meshes/fractal_pad/visual/fractal_L4.stl" />
+        </geometry>
+        <material name="red"/>
+      </visual>
+      <collision>
+        <geometry>
+          <mesh filename="package://fractal_pad_description/meshes/fractal_pad/collision/fractal_L4.stl" />
+        </geometry>
+      </collision>
     </link>
     <link name="${prefix}pad_link">
@@ -35,20 +88,38 @@
       <xacro:insert_block name="origin"/>
       <parent link="${parent}"/>
-      <child link="${prefix}base_link"/>
+      <child link="${prefix}fractal_coupler"/>
     </joint>
-    <joint name="${prefix}motor_joint" type="continuous">
-      <origin xyz="0 0 0.02"/>
-      <parent link="${prefix}base_link"/>
-      <child link="${prefix}motor_link"/>
+    <!-- this here is the moving joint named orignially motor_joint -->
+    <joint name="${prefix}motor_joint" type="fixed">
+      <origin xyz="-0.0354 0 -0.032" rpy="0 0 ${pi/2}"/>
+      <parent link="${prefix}fractal_coupler"/>
+      <child link="${prefix}fractal_L1"/>
+    </joint>
+    <joint name="${prefix}motor_body_joint" type="fixed">
+      <origin xyz="0 -0.025 0" rpy="0 0 ${pi/2}"/>
+      <parent link="${prefix}fractal_L1"/>
+      <child link="${prefix}motor_body"/>
+    </joint>
+    <joint name="${prefix}fractal_L1-fractal_L2_joint" type="revolute">
+      <parent link="${prefix}motor_body"/>
+      <child link="${prefix}fractal_L2"/>
+      <origin xyz="0 0 0" rpy="0 ${-pi/2} 0"/>
       <axis xyz="0 0 1"/>
-      <limit effort="0" velocity="50"/>
+      <limit lower="0" upper="${2*pi}" effort="1" velocity="1"/>
+    </joint>
+      <joint name="${prefix}fractal_L2-fractal_L4_joint" type="revolute">
+      <parent link="${prefix}fractal_L2"/>
+      <child link="${prefix}fractal_L4"/>
+      <origin xyz="0.0095 0 0.008" rpy="0 0 0"/>
+      <axis xyz="0 0 1"/>
+      <limit lower="0" upper="${2*pi}" effort="1" velocity="1"/>
     </joint>
     <joint name="${prefix}motor-pad_joint" type="fixed">
-      <parent link="${prefix}motor_link"/>
+      <parent link="${prefix}fractal_L1"/>
       <child link="${prefix}pad_link"/>
     </joint>
     <joint name="${prefix}pad-tool0_joint" type="fixed">
       <origin xyz="0.115 0 0.08"/>
-      <parent link="${prefix}motor_link"/>
+      <parent link="${prefix}fractal_L1"/>
       <child link="${prefix}tool0"/>
     </joint>

Commit message: Add new links and joints for fractal components in URDF

File: fractal_pad_description/urdf/fractal_pad/fractal_pad_macro.xacro (robot description, xacro)
@@ -75,14 +75,46 @@
       </collision>
     </link>
-    <link name="${prefix}pad_link">
+    <link name="${prefix}fractal_L5325">
       <xacro:default_inertial/>
       <visual>
-        <origin xyz="0.065 0 0.08"/>
-        <geometry><box size="0.10 0.10 0.02"/></geometry>
+        <geometry>
+          <mesh filename="package://fractal_pad_description/meshes/fractal_pad/visual/fractal_L5325-Omega.stl" />
+        </geometry>
         <material name="red"/>
       </visual>
-      <collision><origin xyz="0.065 0 0.08"/><geometry><box size="0.10 0.10 0.02"/></geometry></collision>
+      <collision>
+        <geometry>
+          <mesh filename="package://fractal_pad_description/meshes/fractal_pad/collision/fractal_L5325-Omega.stl" />
+        </geometry>
+      </collision>
     </link>
-    <link name="${prefix}tool0"/>
+    <link name="${prefix}fractal_fingertip_holder">
+      <xacro:default_inertial/>
+      <visual>
+        <geometry>
+          <mesh filename="package://fractal_pad_description/meshes/fractal_pad/visual/fractal_fingertip_holder.stl" />
+        </geometry>
+        <material name="red"/>
+      </visual>
+      <collision>
+        <geometry>
+          <mesh filename="package://fractal_pad_description/meshes/fractal_pad/collision/fractal_fingertip_holder.stl" />
+        </geometry>
+      </collision>
+    </link>
+    <link name="${prefix}fractal_S1813">
+      <xacro:default_inertial/>
+      <visual>
+        <geometry>
+          <mesh filename="package://fractal_pad_description/meshes/fractal_pad/visual/fractal_S1813-Elite.stl" />
+        </geometry>
+        <material name="red"/>
+      </visual>
+      <collision>
+        <geometry>
+          <mesh filename="package://fractal_pad_description/meshes/fractal_pad/collision/fractal_S1813-Elite.stl" />
+        </geometry>
+      </collision>
+    </link>
     <joint name="${prefix}base_joint" type="fixed">
       <xacro:insert_block name="origin"/>
@@ -91,15 +123,15 @@
     </joint>
     <!-- this here is the moving joint named orignially motor_joint -->
-    <joint name="${prefix}motor_joint" type="fixed">
+    <joint name="${prefix}L1_joint" type="fixed">
       <origin xyz="-0.0354 0 -0.032" rpy="0 0 ${pi/2}"/>
       <parent link="${prefix}fractal_coupler"/>
       <child link="${prefix}fractal_L1"/>
     </joint>
-    <joint name="${prefix}motor_body_joint" type="fixed">
+    <joint name="${prefix}L1_motor_body_joint" type="fixed">
       <origin xyz="0 -0.025 0" rpy="0 0 ${pi/2}"/>
       <parent link="${prefix}fractal_L1"/>
       <child link="${prefix}motor_body"/>
     </joint>
-    <joint name="${prefix}fractal_L1-fractal_L2_joint" type="revolute">
+    <joint name="${prefix}L1_L2_joint" type="revolute">
       <parent link="${prefix}motor_body"/>
       <child link="${prefix}fractal_L2"/>
@@ -108,5 +140,5 @@
       <limit lower="0" upper="${2*pi}" effort="1" velocity="1"/>
     </joint>
-      <joint name="${prefix}fractal_L2-fractal_L4_joint" type="revolute">
+      <joint name="${prefix}L2_L4_joint" type="revolute">
       <parent link="${prefix}fractal_L2"/>
       <child link="${prefix}fractal_L4"/>
@@ -115,12 +147,18 @@
       <limit lower="0" upper="${2*pi}" effort="1" velocity="1"/>
     </joint>
-    <joint name="${prefix}motor-pad_joint" type="fixed">
+    <joint name="${prefix}L1_L5325_joint" type="fixed">
+      <origin xyz="0.0051 -0.0637 -0.0362" rpy="0 ${pi} 0"/>
       <parent link="${prefix}fractal_L1"/>
-      <child link="${prefix}pad_link"/>
+      <child link="${prefix}fractal_L5325"/>
     </joint>
-    <joint name="${prefix}pad-tool0_joint" type="fixed">
-      <origin xyz="0.115 0 0.08"/>
-      <parent link="${prefix}fractal_L1"/>
-      <child link="${prefix}tool0"/>
+    <joint name="${prefix}L4_fingertip_holder_joint" type="fixed">
+      <origin xyz="0.0026 -0.0315 0.002" rpy="1 ${pi/2} 0 "/>
+      <parent link="${prefix}fractal_L4"/>
+      <child link="${prefix}fractal_fingertip_holder"/>
+    </joint>
+    <joint name="${prefix}fingertip_holder_S1813_joint" type="fixed">
+      <origin xyz="0.0 0.009 0.0105" rpy="-0.22 0 ${pi}"/>
+      <parent link="${prefix}fractal_fingertip_holder"/>
+      <child link="${prefix}fractal_S1813"/>
     </joint>
   </xacro:macro>

Commit message: Add fractal_L3 link and joint to URDF with visual and collision meshes

File: fractal_pad_description/urdf/fractal_pad/fractal_pad_macro.xacro (robot description, xacro)
@@ -75,4 +75,18 @@
       </collision>
     </link>
+    <link name="${prefix}fractal_L3">
+      <xacro:default_inertial/>
+      <visual>
+        <geometry>
+          <mesh filename="package://fractal_pad_description/meshes/fractal_pad/visual/fractal_L3.stl" />
+        </geometry>
+        <material name="red"/>
+      </visual>
+      <collision>
+        <geometry>
+          <mesh filename="package://fractal_pad_description/meshes/fractal_pad/collision/fractal_L3.stl" />
+        </geometry>
+      </collision>
+    </link>
     <link name="${prefix}fractal_L5325">
       <xacro:default_inertial/>
@@ -147,4 +161,11 @@
       <limit lower="0" upper="${2*pi}" effort="1" velocity="1"/>
     </joint>
+    <joint name="${prefix}L1_L3_joint" type="continuous">
+      <parent link="${prefix}fractal_L1"/>
+      <child link="${prefix}fractal_L3"/>
+      <origin xyz="0 -0.039 -0.022" rpy="${-pi/2} ${-pi/2} 0"/>
+      <axis xyz="0 0 1"/>
+      <limit lower="0" upper="${2*pi}" effort="1" velocity="1"/>
+    </joint>
     <joint name="${prefix}L1_L5325_joint" type="fixed">
       <origin xyz="0.0051 -0.0637 -0.0362" rpy="0 ${pi} 0"/>

Commit message: Add four-bar joint state publisher and update launch files

File: fractal_pad_description/urdf/fractal_pad/fractal_pad_macro.xacro (robot description, xacro)
@@ -25,5 +25,5 @@
           <mesh filename="package://fractal_pad_description/meshes/fractal_pad/visual/fractal_L1.stl" />
         </geometry>
-        <material name="red"/>
+        <material name="white"/>
       </visual>
       <collision>
@@ -39,5 +39,5 @@
           <mesh filename="package://fractal_pad_description/meshes/fractal_pad/visual/fractal_GM2804.stl" />
         </geometry>
-        <material name="grey"/>
+        <material name="black"/>
       </visual>
       <collision>
@@ -53,5 +53,5 @@
           <mesh filename="package://fractal_pad_description/meshes/fractal_pad/visual/fractal_L2.stl" />
         </geometry>
-        <material name="red"/>
+        <material name="grey"/>
       </visual>
       <collision>
@@ -67,5 +67,5 @@
           <mesh filename="package://fractal_pad_description/meshes/fractal_pad/visual/fractal_L4.stl" />
         </geometry>
-        <material name="red"/>
+        <material name="grey"/>
       </visual>
       <collision>
@@ -81,5 +81,5 @@
           <mesh filename="package://fractal_pad_description/meshes/fractal_pad/visual/fractal_L3.stl" />
         </geometry>
-        <material name="red"/>
+        <material name="grey"/>
       </visual>
       <collision>
@@ -95,5 +95,5 @@
           <mesh filename="package://fractal_pad_description/meshes/fractal_pad/visual/fractal_L5325-Omega.stl" />
         </geometry>
-        <material name="red"/>
+        <material name="black"/>
       </visual>
       <collision>
@@ -123,5 +123,5 @@
           <mesh filename="package://fractal_pad_description/meshes/fractal_pad/visual/fractal_S1813-Elite.stl" />
         </geometry>
-        <material name="red"/>
+        <material name="black"/>
       </visual>
       <collision>
@@ -147,15 +147,15 @@
       <child link="${prefix}motor_body"/>
     </joint>
-    <joint name="${prefix}L1_L2_joint" type="revolute">
+    <joint name="${prefix}L1_L2_joint" type="continuous">
       <parent link="${prefix}motor_body"/>
       <child link="${prefix}fractal_L2"/>
       <origin xyz="0 0 0" rpy="0 ${-pi/2} 0"/>
       <axis xyz="0 0 1"/>
-      <limit lower="0" upper="${2*pi}" effort="1" velocity="1"/>
+      <limit lower="${pi/2}" upper="${2*pi}" effort="1" velocity="1"/>
     </joint>
       <joint name="${prefix}L2_L4_joint" type="revolute">
       <parent link="${prefix}fractal_L2"/>
       <child link="${prefix}fractal_L4"/>
-      <origin xyz="0.0095 0 0.008" rpy="0 0 0"/>
+          <origin xyz="0.0095 0 0.009" rpy="0 0 -2.257926628929"/>
       <axis xyz="0 0 1"/>
       <limit lower="0" upper="${2*pi}" effort="1" velocity="1"/>
@@ -164,5 +164,5 @@
       <parent link="${prefix}fractal_L1"/>
       <child link="${prefix}fractal_L3"/>
-      <origin xyz="0 -0.039 -0.022" rpy="${-pi/2} ${-pi/2} 0"/>
+          <origin xyz="0 -0.043 -0.022" rpy="${pi/2} -2.355131484931 0"/>
       <axis xyz="0 0 1"/>
       <limit lower="0" upper="${2*pi}" effort="1" velocity="1"/>

Commit message: added moveit configuration

File: fractal_pad_description/urdf/fractal_pad/fractal_pad_macro.xacro (robot description, xacro)
@@ -3,5 +3,5 @@
   <xacro:include filename="$(find fractal_pad_description)/urdf/common/inertials.xacro" />
   <xacro:include filename="$(find fractal_pad_description)/urdf/common/materials.xacro" />
-  <xacro:macro name="fractal_pad" params="prefix parent *origin">
+  <xacro:macro name="fractal_pad" params="prefix parent planning_mode:=false *origin">
     <!-- Approximate geometry only; replace with measured CAD when available. -->
     <link name="${prefix}fractal_coupler">
@@ -147,25 +147,45 @@
       <child link="${prefix}motor_body"/>
     </joint>
-    <joint name="${prefix}L1_L2_joint" type="continuous">
-      <parent link="${prefix}motor_body"/>
-      <child link="${prefix}fractal_L2"/>
-      <origin xyz="0 0 0" rpy="0 ${-pi/2} 0"/>
-      <axis xyz="0 0 1"/>
-      <limit lower="${pi/2}" upper="${2*pi}" effort="1" velocity="1"/>
-    </joint>
+    <xacro:if value="${planning_mode == True or planning_mode == 'true'}">
+      <!-- Fixed neutral geometry for the seven-joint Panda MoveIt group. -->
+      <joint name="${prefix}L1_L2_joint" type="fixed">
+        <parent link="${prefix}motor_body"/>
+        <child link="${prefix}fractal_L2"/>
+        <origin xyz="0 0 0" rpy="0 ${-pi/2} 0"/>
+      </joint>
+      <joint name="${prefix}L2_L4_joint" type="fixed">
+        <parent link="${prefix}fractal_L2"/>
+        <child link="${prefix}fractal_L4"/>
+        <origin xyz="0.0095 0 0.009" rpy="0 0 -2.257926628929"/>
+      </joint>
+      <joint name="${prefix}L1_L3_joint" type="fixed">
+        <parent link="${prefix}fractal_L1"/>
+        <child link="${prefix}fractal_L3"/>
+        <origin xyz="0 -0.043 -0.022" rpy="${pi/2} -2.355131484931 0"/>
+      </joint>
+    </xacro:if>
+    <xacro:unless value="${planning_mode == True or planning_mode == 'true'}">
+      <joint name="${prefix}L1_L2_joint" type="continuous">
+        <parent link="${prefix}motor_body"/>
+        <child link="${prefix}fractal_L2"/>
+        <origin xyz="0 0 0" rpy="0 ${-pi/2} 0"/>
+        <axis xyz="0 0 1"/>
+        <limit lower="${pi/2}" upper="${2*pi}" effort="1" velocity="1"/>
+      </joint>
       <joint name="${prefix}L2_L4_joint" type="revolute">
-      <parent link="${prefix}fractal_L2"/>
-      <child link="${prefix}fractal_L4"/>
-          <origin xyz="0.0095 0 0.009" rpy="0 0 -2.257926628929"/>
-      <axis xyz="0 0 1"/>
-      <limit lower="0" upper="${2*pi}" effort="1" velocity="1"/>
-    </joint>
-    <joint name="${prefix}L1_L3_joint" type="continuous">
-      <parent link="${prefix}fractal_L1"/>
-      <child link="${prefix}fractal_L3"/>
-          <origin xyz="0 -0.043 -0.022" rpy="${pi/2} -2.355131484931 0"/>
-      <axis xyz="0 0 1"/>
-      <limit lower="0" upper="${2*pi}" effort="1" velocity="1"/>
-    </joint>
+        <parent link="${prefix}fractal_L2"/>
+        <child link="${prefix}fractal_L4"/>
+        <origin xyz="0.0095 0 0.009" rpy="0 0 -2.257926628929"/>
+        <axis xyz="0 0 1"/>
+        <limit lower="0" upper="${2*pi}" effort="1" velocity="1"/>
+      </joint>
+      <joint name="${prefix}L1_L3_joint" type="continuous">
+        <parent link="${prefix}fractal_L1"/>
+        <child link="${prefix}fractal_L3"/>
+        <origin xyz="0 -0.043 -0.022" rpy="${pi/2} -2.355131484931 0"/>
+        <axis xyz="0 0 1"/>
+        <limit lower="0" upper="${2*pi}" effort="1" velocity="1"/>
+      </joint>
+    </xacro:unless>
     <joint name="${prefix}L1_L5325_joint" type="fixed">
       <origin xyz="0.0051 -0.0637 -0.0362" rpy="0 ${pi} 0"/>
